File: hardware/pcb/kicad/mowercarrier.kicad_pcb (KiCad board)
At the start: 2 copper layers, 120 x 100 mm, 49 parts, among them J1 XT60PW-M 12V IN, J2 J_FC: Pixhawk SERVO1/3/6/5, J3 J_5V: servo + ultrasonic, J4 J_M1: IBT-2 #1 (left), J5 J_M2: IBT-2 #2 (right), K1 SLA-12VDC-SL-A DRIVE, K2 SLA-12VDC-SL-A PTO, Q1 IRF4905, Q2 AO3400A, Q3 AO3400A

Commit message: MowerCarrier: Q1 heatsink, 20 A main fuse, zero-warning DRC, deterministic generator
- Q1 heatsink designed in: Fischer SK 104 50,8 STC (9 K/W -> ~46 °C rise at 15 A),
  on the top edge, tied to GND, Q1 on an insulating kit; GND-only pour + no-track zone
  under its fins; power corner re-laid (+12V_IN pour moved to the bottom layer, +12V_RP
  L-pour out of the heatsink mouth, gate network in the mouth, relays down 5 mm)
- F0 30 -> 20 A: the Littelfuse 178.6165.0002 ATO holder is 22.5 A continuous
- DRC: 0 violations of ANY severity (two scoped .kicad_dru exceptions: Q1 inside HS1,
  edge-connector silk), 0 unconnected, parity 0; D1's bus link is a generator-drawn
  locked track; the route is DRC-verified inside the generator and retried
- Deterministic: name-based schematic UUIDs + seeded KiCad KIIDs. Random UUIDs reordered
  the DSN handed to Freerouting, so identical designs routed differently run to run.
  Two full runs now produce a byte-identical .kicad_pcb; check.sh --full gates it
- gen_kicad.sh also exports fab/, schematic.svg, layout.svg and renders from the
  real project; the Rev A concept generators are retired
- check.sh --full: render freshness is perceptual (OpenSCAD anti-aliasing isn't
  bit-stable; a byte diff flagged noise) via scripts/renders_match.py

Co-Authored-By: Claude Opus 5.5 <noreply@anthropic.com>
Parts:
- added HS1: SK 104 50,8 STC 9K/W, Heatsink:Heatsink_Fischer_SK104-STC-STIC_35x13mm_2xDrill2.5mm, F.Cu at (100.0, 57.4)
- F0: value 30A ATO -> 20A ATO (main)
- moved Q1 17.7 mm to (97.5, 61.5)
- moved R1 8.51 mm to (94.5, 67.5), turned to 90 degrees
- moved D5 6.71 mm to (99.0, 65.5), turned to 180 degrees
- moved K1 4.74 mm to (125.5, 78.5)
- moved K2 4.74 mm to (125.5, 118.5)
- moved J2 1.00 mm to (133.0, 112.0)
- moved J3 1.00 mm to (137.0, 112.0)
- moved J4 1.00 mm to (133.0, 90.0)
- moved J5 1.00 mm to (137.0, 90.0)
- moved J1 0.25 mm to (64.0, 66.6)
Routing:
- net /GND: track 594.2 -> 433.0 mm, vias 1 -> 4
- net /+12V_PTO: track 223.4 -> 67.3 mm, vias 1 -> 0
- net /ESTOP_NC1: track 78.9 -> 138.1 mm, vias 1 -> 0
- net /Q1_G: track 29.4 -> 8.14 mm, vias 1 -> 0
- net /DRIVE_EN: track 58.0 -> 74.0 mm
- net /POT_R: track 71.8 -> 86.5 mm
- net /L_REN: track 50.7 -> 37.2 mm
- net /L_RPWM: track 37.9 -> 50.0 mm
- net /MOTOR_V+: track 89.6 -> 77.5 mm
- net /+3V3: track 140.3 -> 131.9 mm
- net /+5V_BUS: track 72.1 -> 64.6 mm
- net /K1_COIL_LO: track 30.6 -> 23.2 mm, vias 2 -> 0
- net /L_LEN: track 47.8 -> 42.8 mm
- net /PTO_OUT: track 36.0 -> 32.4 mm
- net /+12V_DRIVE: track 79.4 -> 76.0 mm, vias 1 -> 0
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- added copper zone on B.Cu, net /+12V_IN
- removed copper zone on F.Cu, net /+12V_IN
