File: hardware/pcb/kicad/mowercarrier.kicad_sch (KiCad schematic)
At the start: 49 parts, among them J1 XT60PW-M 12V IN, J2 J_FC: Pixhawk SERVO1/3/6/5, J3 J_5V: servo + ultrasonic, J4 J_M1: IBT-2 #1 (left), J5 J_M2: IBT-2 #2 (right), K1 SLA-12VDC-SL-A DRIVE, K2 SLA-12VDC-SL-A PTO, Q1 IRF4905, Q2 AO3400A, Q3 AO3400A

Commit message: MowerCarrier: Q1 heatsink, 20 A main fuse, zero-warning DRC, deterministic generator
- Q1 heatsink designed in: Fischer SK 104 50,8 STC (9 K/W -> ~46 °C rise at 15 A),
  on the top edge, tied to GND, Q1 on an insulating kit; GND-only pour + no-track zone
  under its fins; power corner re-laid (+12V_IN pour moved to the bottom layer, +12V_RP
  L-pour out of the heatsink mouth, gate network in the mouth, relays down 5 mm)
- F0 30 -> 20 A: the Littelfuse 178.6165.0002 ATO holder is 22.5 A continuous
- DRC: 0 violations of ANY severity (two scoped .kicad_dru exceptions: Q1 inside HS1,
  edge-connector silk), 0 unconnected, parity 0; D1's bus link is a generator-drawn
  locked track; the route is DRC-verified inside the generator and retried
- Deterministic: name-based schematic UUIDs + seeded KiCad KIIDs. Random UUIDs reordered
  the DSN handed to Freerouting, so identical designs routed differently run to run.
  Two full runs now produce a byte-identical .kicad_pcb; check.sh --full gates it
- gen_kicad.sh also exports fab/, schematic.svg, layout.svg and renders from the
  real project; the Rev A concept generators are retired
- check.sh --full: render freshness is perceptual (OpenSCAD anti-aliasing isn't
  bit-stable; a byte diff flagged noise) via scripts/renders_match.py

Co-Authored-By: Claude Opus 5.5 <noreply@anthropic.com>
Parts:
- added HS1: SK 104 50,8 STC 9K/W, Heatsink:Heatsink_Fischer_SK104-STC-STIC_35x13mm_2xDrill2.5mm, symbol Mechanical:Heatsink_Pad
- F0: value 30A ATO -> 20A ATO (main); LCSC/MPN Littelfuse 178.6165 ATO holder (verify LCSC) -> Littelfuse 178.6165.0002 ATO holder (22.5 A cont.)
- F1, F2, F3, F4, F5: LCSC/MPN Littelfuse 178.6165 ATO holder (verify LCSC) -> Littelfuse 178.6165.0002 ATO holder (22.5 A cont.)
Connections:
- net GND: now also HS1.1
